File: Schematic/Schematic.kicad_sch (KiCad schematic)
At the start: 0 parts

Commit message: Creating the schema for programmer
Parts:
- added C1: 47uF 20v, symbol Device:C_Polarized_Small
- added C2: C_Small, symbol Device:C_Small
- added D1, D2: LED, symbol Device:LED
- added J2: USB, symbol Connector_Generic_MountingPin:Conn_01x04_MountingPin
- added R2, R3, R4: R, symbol Device:R
- added U1: PIC18F2550-ISO, Package_SO:SOIC-28W_7.5x17.9mm_P1.27mm, symbol MCU_Microchip_PIC18:PIC18F2550-ISO
Connections:
- new net: D1.1 (K), R2.1
- new net: R3.2, U1.3 (RA1/AN1)
- new net: D1.2 (A), U1.11 (T1OSO/T13CKI/RC0)
- new net: C1.1, U1.14 (VUSB)
- new net: J2.3 (Pin_3), U1.15 (VM/D-/RC4)
- new net: J2.2 (Pin_2), U1.16 (VP/D+/RC5)
- new net: D2.2 (A), R4.2
- new net +5V: C2.1, J2.1 (Pin_1), R3.1, R4.1, U1.20 (VDD)
- new net GNDREF: C1.2, C2.2, D2.1 (K), J2.4 (Pin_4), R2.2, U1.19 (VSS), U1.8 (VSS)
